File: Kicad/NIVARA/DRY_INPUT_INTERFACE.kicad_sch (KiCad schematic)
At the start: 6 parts, among them U7 LTV-357TB, U8 LTV-357TB

Commit message: Debí de enrutar antes :C
tengo sueño
Parts:
- R11, R13: footprint (none) -> Resistor_SMD:R_0603_1608Metric
Changed lines of the file:
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@@
 			)
 		)
-		(property "Footprint" ""
+		(property "Footprint" "Resistor_SMD:R_0603_1608Metric"
 			(at 138.938 88.9 90)
 			(effects
@@
 			)
 		)
-		(property "Footprint" ""
+		(property "Footprint" "Resistor_SMD:R_0603_1608Metric"
 			(at 138.938 124.46 90)
 			(effects
