File: Kicad/NIVARA/NIVARA_BOARD.kicad_sch (KiCad schematic)
At the start: 3 parts, among them U1 ESP32-S3-WROOM-1

Commit message: ZZZ
Connections:
- net RELAY_INTERFACE/RL1_EN: now also U1.38 (GPIO2/TOUCH2/ADC1_CH1)
- net RELAY_INTERFACE/RL2_EN: now also U1.15 (GPIO3/TOUCH3/ADC1_CH2)
- net mA_INTERFACE_IN/mA_READ: now reaches U1.39 (GPIO1/TOUCH1/ADC1_CH0)
- net mA_INTERFACE_OUT/mA_IN: now reaches U1.4 (GPIO4/TOUCH4/ADC1_CH3)
Other:
- added sheet NPN_IN_Mod (NPN_IN_Mod.kicad_sch)
- added sheet mA_INTERFACE_IN (mA_INTERFACE_IN.kicad_sch)
- added sheet mA_INTERFACE_OUT (mA_INTERFACE.kicad_sch)
- sheet RELAY_INTERFACE ports: added none; removed ST1, ST2

Commit message: .
Parts:
- added R22: R, symbol Device:R
Connections:
- net +3.3V: now also R22.1
- net mA_INTERFACE_OUT/mA_IN: no longer U1.4 (GPIO4/TOUCH4/ADC1_CH3)
- net ~{RUN}/STOP: now also R22.2
Other:
- added sheet 10V_AIN_INTERFACE (10V_AIN_INTERFACE.kicad_sch)
- added sheet 32V_AIN_INTERFACE (32V_AIN_INTERFACE.kicad_sch)
- added sheet DRY_INPUT_INTERFACE (DRY_INPUT_INTERFACE.kicad_sch)
- added sheet NPN_IN_Mod1 (NPN_IN_Mod.kicad_sch)
- added sheet NPN_OUT_INTERFACE (NPN_OUT_INTERFACE.kicad_sch)
- added sheet VOLTAGE_AOUT_INTERFACE (VOLTAGE_AOUT_INTERFACE.kicad_sch)
- sheet NPN_IN_Mod ports: added NPN_Input0, NPN_Input1, NPN_Output0, NPN_Output1; removed none

Commit message: Rutinario
Parts:
- C1: value C -> 1uF
- R1, R22: value R -> 10k
Other:
- removed sheet NPN_IN_Mod1
- added sheet PNP_IN_Mod (PNP_IN_Mod.kicad_sch)
- added sheet PNP_OUT_INTERFACE (PNP_OUT_INTERFACE.kicad_sch)
- sheet DRY_INPUT_INTERFACE ports: added none; removed GND0, GND1

Commit message: FULL SCHEMATIC!!111!!!
Dik
Parts:
- added R31, R32: 4.7k, symbol Device:R
Connections:
- net +3.3V: now also R31.1, R32.1
- net 10V_AIN_INTERFACE/10V_ADC: now also U1.5 (GPIO5/TOUCH5/ADC1_CH4)
- net 32V_AIN_INTERFACE/32V_ADC: now also U1.4 (GPIO4/TOUCH4/ADC1_CH3)
- net DRY_INPUT_INTERFACE/DRY_OUT0: now also U1.18 (GPIO10/TOUCH10/ADC1_CH9/FSPICS0/FSPIIO4/SUBSPICS0)
- net DRY_INPUT_INTERFACE/DRY_OUT1: now also U1.23 (GPIO21)
- net PNP_IN_Mod/NPN_Output0: now also U1.12 (GPIO8/TOUCH8/ADC1_CH7/SUBSPICS1)
- net PNP_IN_Mod/NPN_Output1: now also U1.17 (GPIO9/TOUCH9/ADC1_CH8/FSPIHD/SUBSPIHD)
- net RS485_INTERFACE/UART_RX: now also U1.25 (GPIO48/SPICLK_N/SUBSPICLK_N_DIFF); no longer U1.36 (U0RXD/GPIO44/CLK_OUT2)
- net RS485_INTERFACE/UART_TX: now also U1.24 (GPIO47/SPICLK_P/SUBSPICLK_P_DIFF); no longer U1.37 (U0TXD/GPIO43/CLK_OUT1)
- net RS485_INTERFACE/~{TRANSMIT}/RECEIVE: now also U1.16 (GPIO46)
- net VOLTAGE_AOUT_INTERFACE/SCLK: now also U1.9 (GPIO16/U0CTS/ADC2_CH5/XTAL_32K_N), R31.2, R32.2
- net VOLTAGE_AOUT_INTERFACE/SDA: now also U1.8 (GPIO15/U0RTS/ADC2_CH4/XTAL_32K_P)
- net VOLTAGE_AOUT_INTERFACE/SEL: now also U1.28 (SPIIO6/GPIO35/FSPID/SUBSPID)
- net ~{RUN}/STOP: now also U1.29 (SPIIO7/GPIO36/FSPICLK/SUBSPICLK)
- net NPN_OUT_INTERFACE/NPN_EN1: now reaches U1.26 (GPIO45)
- net NPN_OUT_INTERFACE/NPN_EN0: now reaches U1.31 (GPIO38/FSPIWP/SUBSPIWP)
- net PNP_OUT_INTERFACE/PNP_EN0: now reaches U1.6 (GPIO6/TOUCH6/ADC1_CH5)
- net PNP_OUT_INTERFACE/PNP_EN1: now reaches U1.7 (GPIO7/TOUCH7/ADC1_CH6)
Other:
- sheet NPN_OUT_INTERFACE ports: added NPN_EN0, NPN_EN1; removed NPN_OUT_EN0, NPN_OUT_EN1
- sheet PNP_OUT_INTERFACE ports: added PNP_EN0, PNP_EN1; removed none
- sheet mA_INTERFACE_OUT ports: added SCLK, SDA; removed mA_IN, mA_OUT-
- moved on the sheet: C1, R1, R22, U1
