File: Kicad/NIVARA/NIVARA_BOARD.kicad_sch (KiCad schematic)
At the start: 6 parts, among them U1 ESP32-S3-WROOM-1

Commit message: Commit
Connections:
- net NPN_IN_Mod/NPN_Output0: now also U1.19 (GPIO11/TOUCH11/ADC2_CH0/FSPID/FSPIIO5/SUBSPID)
- net NPN_IN_Mod/NPN_Output1: now also U1.20 (GPIO12/TOUCH12/ADC2_CH1/FSPICLK/FSPIIO6/SUBSPICLK)
- net RS485_INTERFACE/~{TRANSMIT}/RECEIVE renamed RS485_INTERFACE/~{TX}/RX
Other:
- sheet RS485_INTERFACE ports: added ~{TX}/RX; removed ~{TRANSMIT}/RECEIVE
Changed lines of the file:
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@@
+	(wire
+		(pts
+			(xy 267.97 170.18) (xy 267.97 87.63)
+		)
+		(stroke
+			(width 0)
+			(type default)
+		)
+	)
 	(wire
 		(pts
@@
 	(wire
 		(pts
+			(xy 290.83 176.53) (xy 265.43 176.53)
+		)
+		(stroke
+			(width 0)
+			(type default)
+		)
+	)
+	(wire
+		(pts
 			(xy 290.83 72.39) (xy 288.29 72.39)
 		)
@@
 	(wire
 		(pts
+			(xy 267.97 87.63) (xy 260.35 87.63)
+		)
+		(stroke
+			(width 0)
+			(type default)
+		)
+	)
+	(wire
+		(pts
 			(xy 281.94 137.16) (xy 290.83 137.16)
 		)
@@
 	(wire
 		(pts
+			(xy 265.43 90.17) (xy 260.35 90.17)
+		)
+		(stroke
+			(width 0)
+			(type default)
+		)
+	)
+	(wire
+		(pts
 			(xy 290.83 124.46) (xy 283.21 124.46)
 		)
@@
 	(wire
 		(pts
+			(xy 265.43 176.53) (xy 265.43 90.17)
+		)
+		(stroke
+			(width 0)
+			(type default)
+		)
+	)
+	(wire
+		(pts
 			(xy 260.35 107.95) (xy 273.05 107.95)
 		)
@@
 	(wire
 		(pts
-			(xy 269.24 110.49) (xy 260.35 110.49)
-		)
-		(stroke
-			(width 0)
-			(type default)
-		)
-	)
-	(wire
-		(pts
 			(xy 325.12 124.46) (xy 321.31 124.46)
 		)
@@
 	(wire
 		(pts
+			(xy 260.35 110.49) (xy 269.24 110.49)
+		)
+		(stroke
+			(width 0)
+			(type default)
+		)
+	)
+	(wire
+		(pts
 			(xy 320.04 190.5) (xy 316.23 190.5)
 		)
@@
 	(wire
 		(pts
+			(xy 290.83 170.18) (xy 267.97 170.18)
+		)
+		(stroke
+			(width 0)
+			(type default)
+		)
+	)
+	(wire
+		(pts
 			(xy 147.32 39.37) (xy 151.13 39.37)
 		)
@@
 	(wire
 		(pts
+			(xy 269.24 229.87) (xy 290.83 229.87)
+		)
+		(stroke
+			(width 0)
+			(type default)
+		)
+	)
+	(wire
+		(pts
 			(xy 139.7 52.07) (xy 139.7 44.45)
 		)
@@
 		(pts
 			(xy 323.85 87.63) (xy 327.66 87.63)
-		)
-		(stroke
-			(width 0)
-			(type default)
-		)
-	)
-	(wire
-		(pts
-			(xy 290.83 229.87) (xy 269.24 229.87)
 		)
 		(stroke
@@
 			)
 		)
-		(pin "~{TRANSMIT}{slash}RECEIVE" input
+		(pin "~{TX}{slash}RX" input
 			(at 290.83 229.87 180)
 			(effects

Commit message: Faltan dos Cositas
Casi terminamos de enrutar
Connections:
- net VOLTAGE_AOUT_INTERFACE/SCLK: no longer R32.2
- net VOLTAGE_AOUT_INTERFACE/SDA: now also R32.2
Changed lines of the file:
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@@
-	)
-	(junction
-		(at 151.13 54.61)
-		(diameter 0)
-		(color 0 0 0 0)
 	)
 	(junction
@@
 		(color 0 0 0 0)
 	)
+	(junction
+		(at 151.13 52.07)
+		(diameter 0)
+		(color 0 0 0 0)
+	)
 	(wire
 		(pts
@@
 	(wire
 		(pts
-			(xy 143.51 54.61) (xy 151.13 54.61)
+			(xy 151.13 50.8) (xy 151.13 52.07)
+		)
+		(stroke
+			(width 0)
+			(type default)
+		)
+	)
+	(wire
+		(pts
+			(xy 143.51 54.61) (xy 168.91 54.61)
 		)
 		(stroke
@@
 	(wire
 		(pts
+			(xy 151.13 52.07) (xy 168.91 52.07)
+		)
+		(stroke
+			(width 0)
+			(type default)
+		)
+	)
+	(wire
+		(pts
 			(xy 260.35 77.47) (xy 280.67 77.47)
 		)
@@
 	(wire
 		(pts
-			(xy 151.13 50.8) (xy 151.13 54.61)
-		)
-		(stroke
-			(width 0)
-			(type default)
-		)
-	)
-	(wire
-		(pts
 			(xy 260.35 102.87) (xy 275.59 102.87)
 		)
@@
 	(wire
 		(pts
-			(xy 139.7 52.07) (xy 168.91 52.07)
+			(xy 139.7 52.07) (xy 151.13 52.07)
 		)
 		(stroke
@@
 		)
 		(stroke
-			(width 0)
-			(type default)
-		)
-	)
-	(wire
-		(pts
-			(xy 151.13 54.61) (xy 168.91 54.61)
-		)
-		(stroke
