File: Kicad/NIVARA/NIVARA.kicad_sch (KiCad schematic)
At the start: 0 parts

Commit message: Hierarchical Design In KiCAD
Parts:
- added J1: Screw_Terminal_01x02, symbol Connector:Screw_Terminal_01x02
Other:
- added sheet NIVARA_BOARD (NIVARA_BOARD.kicad_sch)
Changed lines of the file:
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@@
 	(generator_version "9.0")
 	(paper "A4")
+	(symbol
+		(lib_id "Connector:Screw_Terminal_01x02")
+		(at 95.25 53.34 0)
+		(mirror y)
+		(unit 1)
+		(exclude_from_sim no)
+		(in_bom yes)
+		(on_board yes)
+		(dnp no)
+		(fields_autoplaced yes)
+		(property "Reference" "J1"
+			(at 95.25 46.99 0)
+			(effects
+				(font
+					(size 1.27 1.27)
+				)
+			)
+		)
+		(property "Value" "Screw_Terminal_01x02"
+			(at 95.25 49.53 0)
+			(effects
+				(font
+					(size 1.27 1.27)
+				)
+			)
+		)
+		(property "Footprint" ""
+			(at 95.25 53.34 0)
+			(effects
+				(font
+					(size 1.27 1.27)
+				)
+				(hide yes)
+			)
+		)
+		(property "Datasheet" "~"
+			(at 95.25 53.34 0)
+			(effects
+				(font
+					(size 1.27 1.27)
+				)
+				(hide yes)
+			)
+		)
+		(property "Description" "Generic screw terminal, single row, 01x02, script generated (kicad-library-utils/schlib/autogen/connector/)"
+			(at 95.25 53.34 0)
+			(effects
+				(font
+					(size 1.27 1.27)
+				)
+				(hide yes)
+			)
+		)
+		(pin "2"
+		)
+		(pin "1"
+		)
+		(instances
+			(project ""
+				(path "/8290cc18-06d0-4e02-a781-29a61ebc321a"
+					(reference "J1")
+					(unit 1)
+				)
+			)
+		)
+	)
+	(sheet
+		(at 114.3 45.72)
+		(size 67.31 55.88)
+		(exclude_from_sim no)
+		(in_bom yes)
+		(on_board yes)
+		(dnp no)
+		(fields_autoplaced yes)
+		(stroke
+			(width 0.1524)
+			(type solid)
+		)
+		(fill
+			(color 0 0 0 0.0000)
+		)
+		(property "Sheetname" "NIVARA_BOARD"
+			(at 114.3 45.0084 0)
+			(effects
+				(font
+					(size 1.27 1.27)
+				)
+				(justify left bottom)
+			)
+		)
+		(property "Sheetfile" "NIVARA_BOARD.kicad_sch"
+			(at 114.3 102.1846 0)
+			(effects
+				(font
+					(size 1.27 1.27)
+				)
+				(justify left top)
+			)
+		)
+		(instances
+			(project "NIVARA"
+				(path "/8290cc18-06d0-4e02-a781-29a61ebc321a"
+					(page "2")
+				)
+			)
+		)
+	)
 	(sheet_instances
 		(path "/"

Commit message: Initial Capture Finished
Parts:
- added J10, J2, J4, J5, J9: Screw_Terminal_01x02, symbol Connector:Screw_Terminal_01x02
- added J3: Screw_Terminal_01x04, symbol Connector:Screw_Terminal_01x04
- added J6: Screw_Terminal_01x06, symbol Connector:Screw_Terminal_01x06
- added J7, J8: Screw_Terminal_01x03, symbol Connector:Screw_Terminal_01x03
Connections:
- net NIVARA_BOARD/NPN_DINPUT_0: now reaches J1.1 (Pin_1)
- net NIVARA_BOARD/NPN_DINPUT_1: now reaches J1.2 (Pin_2)
- new net GND: J3.4 (Pin_4), J5.2 (Pin_2), J7.3 (Pin_3), J8.3 (Pin_3)
- new net NIVARA_BOARD/+10V_AINPUT: J3.1 (Pin_1)
- new net NIVARA_BOARD/+32V_AINPUT: J3.2 (Pin_2)
- new net NIVARA_BOARD/NPN_DOUTPUT_0: J9.1 (Pin_1)
- new net NIVARA_BOARD/NPN_DOUTPUT_1: J9.2 (Pin_2)
- new net NIVARA_BOARD/OPTO_DINPUT_0: J4.1 (Pin_1)
- new net NIVARA_BOARD/OPTO_DINPUT_1: J4.2 (Pin_2)
- new net NIVARA_BOARD/PNP_DINPUT_0: J2.1 (Pin_1)
- new net NIVARA_BOARD/PNP_DINPUT_1: J2.2 (Pin_2)
- new net NIVARA_BOARD/PNP_DOUTPUT_0: J10.1 (Pin_1)
- new net NIVARA_BOARD/PNP_DOUTPUT_1: J10.2 (Pin_2)
- new net NIVARA_BOARD/RL1_COM: J6.3 (Pin_3)
- new net NIVARA_BOARD/RL1_OUTPUT_NC: J6.2 (Pin_2)
- new net NIVARA_BOARD/RL1_OUTPUT_NO: J6.1 (Pin_1)
- new net NIVARA_BOARD/RL2_COM: J6.6 (Pin_6)
- new net NIVARA_BOARD/RL2_OUTPUT_NC: J6.5 (Pin_5)
- new net NIVARA_BOARD/RL2_OUTPUT_NO: J6.4 (Pin_4)
- new net NIVARA_BOARD/RS485_A: J7.1 (Pin_1)
- new net NIVARA_BOARD/RS485_B: J7.2 (Pin_2)
- new net NIVARA_BOARD/VOLTAGE_AOUTPUT: J8.1 (Pin_1)
- new net NIVARA_BOARD/mA_AINPUT: J3.3 (Pin_3)
- new net NIVARA_BOARD/mA_AOUTPUT: J8.2 (Pin_2)
- new net NIVARA_BOARD/~{RUN}/STOP: J5.1 (Pin_1)
Other:
- sheet NIVARA_BOARD ports: added +10V_AINPUT, +32V_AINPUT, NPN_DINPUT_0, NPN_DINPUT_1, NPN_DOUTPUT_0, NPN_DOUTPUT_1, OPTO_DINPUT_0, OPTO_DINPUT_1, PNP_DINPUT_0, PNP_DINPUT_1, PNP_DOUTPUT_0, PNP_DOUTPUT_1, RL1_COM, RL1_OUTPUT_NC, RL1_OUTPUT_NO, RL2_COM, RL2_OUTPUT_NC, RL2_OUTPUT_NO, RS485_A, RS485_B, VOLTAGE_AOUTPUT, mA_AINPUT, mA_AOUTPUT, ~{RUN}/STOP; removed none
- moved on the sheet: J1

Commit message: Wrapping up for today :3
Parts:
- added AE1: WIFI-BT, symbol Device:Antenna
- added J11: Screw_Terminal_01x02, symbol Connector:Screw_Terminal_01x02
Connections:
- net GND: now also J11.2 (Pin_2)
- new net VCC: J11.1 (Pin_1)
Other:
- note added: "+24VDC"

Commit message: ZZZ
Parts:
- AE1: value WIFI-BT -> Antenna
Changed lines of the file:
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@@
 		(dnp no)
 		(fields_autoplaced yes)
-		(property "Reference" "#PWR07"
+		(property "Reference" "#PWR7"
 			(at 140.97 30.48 0)
 			(effects
@@
 			(project ""
 				(path "/8290cc18-06d0-4e02-a781-29a61ebc321a"
-					(reference "#PWR07")
+					(reference "#PWR7")
 					(unit 1)
 				)
@@
 		(dnp no)
 		(fields_autoplaced yes)
-		(property "Reference" "#PWR05"
+		(property "Reference" "#PWR5"
 			(at 184.15 63.5 0)
 			(effects
@@
 			(project "NIVARA"
 				(path "/8290cc18-06d0-4e02-a781-29a61ebc321a"
-					(reference "#PWR05")
+					(reference "#PWR5")
 					(unit 1)
 				)
@@
 		(dnp no)
 		(fields_autoplaced yes)
-		(property "Reference" "#PWR03"
+		(property "Reference" "#PWR3"
 			(at 111.76 87.63 0)
 			(effects
@@
 			(project "NIVARA"
 				(path "/8290cc18-06d0-4e02-a781-29a61ebc321a"
-					(reference "#PWR03")
+					(reference "#PWR3")
 					(unit 1)
 				)
@@
 		(dnp no)
 		(fields_autoplaced yes)
-		(property "Reference" "#PWR06"
+		(property "Reference" "#PWR6"
 			(at 140.97 38.1 0)
 			(effects
@@
 			(project ""
 				(path "/8290cc18-06d0-4e02-a781-29a61ebc321a"
-					(reference "#PWR06")
+					(reference "#PWR6")
 					(unit 1)
 				)
@@
 		(dnp no)
 		(fields_autoplaced yes)
-		(property "Reference" "#PWR04"
+		(property "Reference" "#PWR4"
 			(at 184.15 53.34 0)
 			(effects
@@
 			(project "NIVARA"
 				(path "/8290cc18-06d0-4e02-a781-29a61ebc321a"
-					(reference "#PWR04")
+					(reference "#PWR4")
 					(unit 1)
 				)
@@
 		(dnp no)
 		(fields_autoplaced yes)
-		(property "Reference" "#PWR02"
+		(property "Reference" "#PWR2"
 			(at 111.76 72.39 0)
 			(effects
@@
 			(project ""
 				(path "/8290cc18-06d0-4e02-a781-29a61ebc321a"
-					(reference "#PWR02")
+					(reference "#PWR2")
 					(unit 1)
 				)
@@
 			)
 		)
-		(property "Value" "WIFI-BT"
+		(property "Value" "Antenna"
 			(at 161.29 32.3849 0)
 			(effects

Commit message: Rutinario
Parts:
- removed J8: Screw_Terminal_01x03, symbol Connector:Screw_Terminal_01x03
- added J12: Screw_Terminal_01x04, symbol Connector:Screw_Terminal_01x04
Connections:
- net GND: now also J12.4 (Pin_4)
- net NIVARA_BOARD/VOLTAGE_AOUTPUT: now also J12.1 (Pin_1)
- net NIVARA_BOARD/OPTO_DINPUT_0 renamed NIVARA_BOARD/DRY_DINPUT_0
- net NIVARA_BOARD/OPTO_DINPUT_1 renamed NIVARA_BOARD/DRY_DINPUT_1
- new net NIVARA_BOARD/mA_AOUTPUT+: J12.2 (Pin_2)
- new net NIVARA_BOARD/mA_AOUTPUT-: J12.3 (Pin_3)
Other:
- sheet NIVARA_BOARD ports: added DRY_DINPUT_0, DRY_DINPUT_1, mA_AOUTPUT+, mA_AOUTPUT-; removed OPTO_DINPUT_0, OPTO_DINPUT_1, mA_AOUTPUT
- moved on the sheet: J10, J6, J9

Commit message: FULL SCHEMATIC!!111!!!
Dik
Parts:
- removed J1, J10, J2, J4, J9: Screw_Terminal_01x02, symbol Connector:Screw_Terminal_01x02
- added J1, J2, J4, J8, J9: Screw_Terminal_01x03, symbol Connector:Screw_Terminal_01x03
Connections:
- net GND: now also J4.3 (Pin_3), J9.1 (Pin_1)
- net NIVARA_BOARD/DRY_DINPUT_0: now also J4.1 (Pin_1)
- net NIVARA_BOARD/DRY_DINPUT_1: now also J4.2 (Pin_2)
- net NIVARA_BOARD/NPN_DINPUT_0: now also J1.1 (Pin_1)
- net NIVARA_BOARD/NPN_DINPUT_1: now also J1.2 (Pin_2)
- net NIVARA_BOARD/NPN_DOUTPUT_0: now also J8.2 (Pin_2)
- net NIVARA_BOARD/NPN_DOUTPUT_1: now also J8.3 (Pin_3)
- net NIVARA_BOARD/PNP_DINPUT_0: now also J2.1 (Pin_1)
- net NIVARA_BOARD/PNP_DINPUT_1: now also J2.2 (Pin_2)
- net NIVARA_BOARD/PNP_DOUTPUT_0: now also J9.2 (Pin_2)
- net NIVARA_BOARD/PNP_DOUTPUT_1: now also J9.3 (Pin_3)
- net VCC: now also J8.1 (Pin_1)
- net NIVARA_BOARD/mA_AOUTPUT-: no longer names the net of J12.3 (Pin_3)
- new net NPNIN_GND: J1.3 (Pin_3)
- new net PNPIN_GND: J2.3 (Pin_3)
Other:
- sheet NIVARA_BOARD ports: added none; removed mA_AOUTPUT-
- moved on the sheet: J3, J5

Commit message: Debí de enrutar antes :C
tengo sueño
Parts:
- J1, J2, J4, J7, J8, J9: footprint (none) -> TerminalBlock_4Ucon:TerminalBlock_4Ucon_1x03_P3.50mm_Horizontal
- J11, J5: footprint (none) -> TerminalBlock_4Ucon:TerminalBlock_4Ucon_1x02_P3.50mm_Horizontal
- J12, J3: footprint (none) -> TerminalBlock_4Ucon:TerminalBlock_4Ucon_1x04_P3.50mm_Horizontal
- J6: footprint (none) -> TerminalBlock_4Ucon:TerminalBlock_4Ucon_1x06_P3.50mm_Horizontal
Changed lines of the file:
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@@
 			)
 		)
-		(property "Footprint" ""
+		(property "Footprint" "TerminalBlock_4Ucon:TerminalBlock_4Ucon_1x04_P3.50mm_Horizontal"
 			(at 198.12 60.96 0)
 			(effects
@@
 			)
 		)
-		(property "Footprint" ""
+		(property "Footprint" "TerminalBlock_4Ucon:TerminalBlock_4Ucon_1x03_P3.50mm_Horizontal"
 			(at 198.12 102.87 0)
 			(effects
@@
 			)
 		)
-		(property "Footprint" ""
+		(property "Footprint" "TerminalBlock_4Ucon:TerminalBlock_4Ucon_1x06_P3.50mm_Horizontal"
 			(at 198.12 77.47 0)
 			(effects
@@
 			)
 		)
-		(property "Footprint" ""
+		(property "Footprint" "TerminalBlock_4Ucon:TerminalBlock_4Ucon_1x02_P3.50mm_Horizontal"
 			(at 91.44 92.71 0)
 			(effects
@@
 			)
 		)
-		(property "Footprint" ""
+		(property "Footprint" "TerminalBlock_4Ucon:TerminalBlock_4Ucon_1x03_P3.50mm_Horizontal"
 			(at 91.44 52.07 0)
 			(effects
@@
 			)
 		)
-		(property "Footprint" ""
+		(property "Footprint" "TerminalBlock_4Ucon:TerminalBlock_4Ucon_1x04_P3.50mm_Horizontal"
 			(at 91.44 72.39 0)
 			(effects
@@
 			)
 		)
-		(property "Footprint" ""
+		(property "Footprint" "TerminalBlock_4Ucon:TerminalBlock_4Ucon_1x03_P3.50mm_Horizontal"
 			(at 91.44 62.23 0)
 			(effects
@@
 			)
 		)
-		(property "Footprint" ""
+		(property "Footprint" "TerminalBlock_4Ucon:TerminalBlock_4Ucon_1x02_P3.50mm_Horizontal"
 			(at 134.62 27.94 0)
 			(effects
@@
 			)
 		)
-		(property "Footprint" ""
+		(property "Footprint" "TerminalBlock_4Ucon:TerminalBlock_4Ucon_1x03_P3.50mm_Horizontal"
 			(at 198.12 50.8 0)
 			(effects
@@
 			)
 		)
-		(property "Footprint" ""
+		(property "Footprint" "TerminalBlock_4Ucon:TerminalBlock_4Ucon_1x03_P3.50mm_Horizontal"
 			(at 198.12 92.71 0)
 			(effects
@@
 			)
 		)
-		(property "Footprint" ""
+		(property "Footprint" "TerminalBlock_4Ucon:TerminalBlock_4Ucon_1x03_P3.50mm_Horizontal"
 			(at 91.44 85.09 0)
 			(effects
