File: Kicad/NIVARA/NIVARA.kicad_sch (KiCad schematic)
At the start: 12 parts, among them J1 Screw_Terminal_01x03, J11 Screw_Terminal_01x02, J12 Screw_Terminal_01x04, J2 Screw_Terminal_01x03, J3 Screw_Terminal_01x04, J4 Screw_Terminal_01x03, J5 Screw_Terminal_01x02, J6 Screw_Terminal_01x06, J7 Screw_Terminal_01x03, J8 Screw_Terminal_01x03, J9 Screw_Terminal_01x03

Commit message: Faltan dos Cositas
Casi terminamos de enrutar
Connections:
- net NIVARA_BOARD/RL1_COM: now also J6.2 (Pin_2); no longer J6.3 (Pin_3)
- net NIVARA_BOARD/RL1_OUTPUT_NC: now also J6.3 (Pin_3); no longer J6.2 (Pin_2)
- net NIVARA_BOARD/RL2_COM: now also J6.5 (Pin_5); no longer J6.6 (Pin_6)
- net NIVARA_BOARD/RL2_OUTPUT_NC: now also J6.6 (Pin_6); no longer J6.5 (Pin_5)
Changed lines of the file:
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@@
 	(wire
 		(pts
-			(xy 181.61 74.93) (xy 193.04 74.93)
+			(xy 181.61 77.47) (xy 193.04 77.47)
 		)
 		(stroke
@@
 	(wire
 		(pts
-			(xy 96.52 95.25) (xy 99.06 95.25)
+			(xy 181.61 74.93) (xy 193.04 74.93)
 		)
 		(stroke
@@
 	(wire
 		(pts
-			(xy 96.52 87.63) (xy 99.06 87.63)
+			(xy 96.52 95.25) (xy 99.06 95.25)
 		)
 		(stroke
@@
 	(wire
 		(pts
-			(xy 139.7 27.94) (xy 140.97 27.94)
+			(xy 96.52 87.63) (xy 99.06 87.63)
 		)
 		(stroke
@@
 	(wire
 		(pts
-			(xy 181.61 58.42) (xy 193.04 58.42)
+			(xy 139.7 27.94) (xy 140.97 27.94)
 		)
 		(stroke
@@
 	(wire
 		(pts
-			(xy 181.61 50.8) (xy 193.04 50.8)
+			(xy 181.61 58.42) (xy 193.04 58.42)
 		)
 		(stroke
@@
 	(wire
 		(pts
-			(xy 181.61 77.47) (xy 193.04 77.47)
+			(xy 181.61 50.8) (xy 193.04 50.8)
 		)
 		(stroke
@@
 	(wire
 		(pts
-			(xy 181.61 82.55) (xy 193.04 82.55)
+			(xy 139.7 30.48) (xy 140.97 30.48)
 		)
 		(stroke
@@
 	(wire
 		(pts
-			(xy 139.7 30.48) (xy 140.97 30.48)
+			(xy 96.52 92.71) (xy 114.3 92.71)
 		)
 		(stroke
@@
 	(wire
 		(pts
-			(xy 96.52 92.71) (xy 114.3 92.71)
+			(xy 96.52 77.47) (xy 99.06 77.47)
 		)
 		(stroke
@@
 	(wire
 		(pts
-			(xy 96.52 77.47) (xy 99.06 77.47)
+			(xy 181.61 95.25) (xy 193.04 95.25)
 		)
 		(stroke
@@
 	(wire
 		(pts
-			(xy 181.61 95.25) (xy 193.04 95.25)
+			(xy 181.61 82.55) (xy 193.04 82.55)
 		)
 		(stroke
@@
 		)
 		(pin "RL1_COM" passive
-			(at 181.61 77.47 0)
+			(at 181.61 74.93 0)
 			(effects
 				(font
@@
 		)
 		(pin "RL1_OUTPUT_NC" output
-			(at 181.61 74.93 0)
+			(at 181.61 77.47 0)
 			(effects
 				(font
@@
 		)
 		(pin "RL2_COM" passive
-			(at 181.61 85.09 0)
+			(at 181.61 82.55 0)
 			(effects
 				(font
@@
 		)
 		(pin "RL2_OUTPUT_NC" output
-			(at 181.61 82.55 0)
+			(at 181.61 85.09 0)
 			(effects
 				(font
