File: Kicad/NIVARA/PNP_OUT_INTERFACE.kicad_sch (KiCad schematic)
At the start: 8 parts, among them Q1 NCV8402xST, Q3 NCV8402xST, U12 LTV-357T, U5 LTV-357T

Commit message: Rutinario
Parts:
- removed Q1, Q3: NCV8402xST, Package_TO_SOT_SMD:SOT-223, symbol Driver_FET:NCV8402xST
- removed R26, R27: 100, symbol Device:R
- removed R28, R4: R, symbol Device:R
- removed U12, U5: LTV-357T, Package_SO:SO-4_4.4x3.6mm_P2.54mm, symbol Isolator:LTV-357T
- added Q4, Q5: NCV8402xST, Package_TO_SOT_SMD:SOT-223, symbol Driver_FET:NCV8402xST
- added R29, R31: 100, symbol Device:R
- added R30, R32: R, symbol Device:R
- added U13, U14: LTV-357T, Package_SO:SO-4_4.4x3.6mm_P2.54mm, symbol Isolator:LTV-357T
Connections:
- net GND: now also U13.2, U14.2
- new net: Q5.1 (G), R32.1, U14.3
- new net: R31.2, U14.1
- new net: R29.2, U13.1
- new net PNPOUT_GND: Q4.3 (S), Q5.3 (S), R32.2, U13.3
- new net PNP_OUT0: Q4.2 (D), Q4.4 (D)
- new net PNP_OUT1: Q5.2 (D), Q5.4 (D)
- new net PNP_VCC: U14.4

Commit message: FULL SCHEMATIC!!111!!!
Dik
Parts:
- removed Q4, Q5: NCV8402xST, Package_TO_SOT_SMD:SOT-223, symbol Driver_FET:NCV8402xST
- removed R31: 100, symbol Device:R
- removed R32: R, symbol Device:R
- removed U13, U14: LTV-357T, Package_SO:SO-4_4.4x3.6mm_P2.54mm, symbol Isolator:LTV-357T
- added U13, U14: ~, Package_SO:SO-4_4.4x4.3mm_P2.54mm, symbol Riqi_Parts:GAQY211G2S
- R30: value R -> 100
Connections:
- net GND: now also U13.2, U14.2
- net PNP_OUT0: now also U13.4
- net PNP_OUT1: now also U14.4
- net PNP_EN1: now reaches R30.1
- net at R30.2: now also U14.1
- net PNP_EN0: now reaches R29.1
- net at R29.2: now also U13.1
- new net VCC: U13.3, U14.3

Commit message: Debí de enrutar antes :C
tengo sueño
Parts:
- R29, R30: footprint (none) -> Resistor_SMD:R_0603_1608Metric
Changed lines of the file:
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@@
 			)
 		)
-		(property "Footprint" ""
+		(property "Footprint" "Resistor_SMD:R_0603_1608Metric"
 			(at 125.73 94.488 90)
 			(effects
@@
 			)
 		)
-		(property "Footprint" ""
+		(property "Footprint" "Resistor_SMD:R_0603_1608Metric"
 			(at 64.77 94.488 90)
 			(effects
