File: Kicad/NIVARA/RS485_INTERFACE.kicad_sch (KiCad schematic)
At the start: 4 parts

Commit message: Debí de enrutar antes :C
tengo sueño
Parts:
- R24, R25: footprint (none) -> Resistor_SMD:R_0603_1608Metric
Changed lines of the file:
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@@
 			)
 		)
-		(property "Footprint" ""
+		(property "Footprint" "Resistor_SMD:R_0603_1608Metric"
 			(at 142.24 72.898 90)
 			(effects
@@
 			)
 		)
-		(property "Footprint" ""
+		(property "Footprint" "Resistor_SMD:R_0603_1608Metric"
 			(at 142.24 73.152 90)
 			(effects
