File: Kicad/NIVARA/mA_INTERFACE.kicad_sch (KiCad schematic)
At the start: 4 parts, among them U6 XTR116U

Commit message: .
Parts:
- removed C7: C, symbol Device:C
- removed R7: R, symbol Device:R

Commit message: Rutinario
Parts:
- removed U6: XTR116U, Package_SO:SOIC-8_3.9x4.9mm_P1.27mm, symbol Interface_CurrentLoop:XTR116U
- added C12: 220pF, symbol Device:C
- added C13: 1uF, symbol Device:C
- added D1: D_Zener, symbol Device:D_Zener
- added JP2, JP3, JP4: SolderJumper_2_Open, symbol Jumper:SolderJumper_2_Open
- added R33, R34, R35: 10k, symbol Device:R
- added U6: ~, Package_SO:SSOP-10-1EP_3.9x4.9mm_P1mm_EP2.1x3.3mm, symbol Riqi_Parts:GP8303
- R6: value R -> 2.5k
Connections:
- net GND: now also R6.2, C12.2, C13.2, JP2.1 (A), JP3.1 (A), JP4.1 (A), U6.6 (GND)
- net VCC: now also D1.1 (K), U6.5 (VCC)
- net at R6.1: now also C12.1, U6.7 (SET)
- new net: C13.1, R33.1, R34.1, R35.1, U6.10 (V5V)
- new net: JP2.2 (B), R33.2, U6.3 (A0)
- new net: JP3.2 (B), R34.2, U6.4 (A1)
- new net: JP4.2 (B), R35.2, U6.9 (A2)
- no-connect marks 2 -> 0

Commit message: FULL SCHEMATIC!!111!!!
Dik
Parts:
- added C14: 1uF, symbol Device:C
- added C15: 100nF, symbol Device:C
- added D4: 1N4007, Diode_THT:D_DO-41_SOD81_P10.16mm_Horizontal, symbol Diode:1N4007
- added D5: SMF24A, Diode_SMD:D_SMF, symbol Diode:SMF24A
- added R27: 100k, symbol Device:R
- added R28: 15, symbol Device:R
- added T1: IRF9310TRPBF, IRF9310TRPBF:SO-8, symbol Riqi_Parts:IRF9310TRPBF
Connections:
- net GND: now also C14.2, C15.2, D5.2 (A2), R27.2
- net mA_OUT+: now also D4.1 (K)
- net SCLK: now reaches U6.1 (SCLK)
- net SDA: now reaches U6.2 (SDA)
- net at U6.8 (IOUT): now also T1.1, T1.2, T1.3
- net at D1.2 (A): now also C14.1, R27.1, T1.4
- new net: C15.1, D5.1 (A1), R28.1, T1.5, T1.6, T1.7, T1.8
- new net: D4.2 (A), R28.2
Other:
- moved on the sheet: D1

Commit message: Debí de enrutar antes :C
tengo sueño
Parts:
- C12, C13, C14, C15: footprint (none) -> Capacitor_SMD:C_0603_1608Metric
- JP2, JP3, JP4: footprint (none) -> Jumper:SolderJumper-2_P1.3mm_Open_RoundedPad1.0x1.5mm
- R27, R28, R33, R34, R35, R6: footprint (none) -> Resistor_SMD:R_0603_1608Metric
Changed lines of the file:
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@@
 			)
 		)
-		(property "Footprint" ""
+		(property "Footprint" "Resistor_SMD:R_0603_1608Metric"
 			(at 154.432 104.14 90)
 			(effects
@@
 			)
 		)
-		(property "Footprint" ""
+		(property "Footprint" "Capacitor_SMD:C_0603_1608Metric"
 			(at 222.5548 111.76 0)
 			(effects
@@
 			)
 		)
-		(property "Footprint" ""
+		(property "Footprint" "Resistor_SMD:R_0603_1608Metric"
 			(at 236.22 105.918 90)
 			(effects
@@
 			)
 		)
-		(property "Footprint" ""
+		(property "Footprint" "Resistor_SMD:R_0603_1608Metric"
 			(at 120.65 98.298 90)
 			(effects
@@
 			)
 		)
-		(property "Footprint" ""
+		(property "Footprint" "Capacitor_SMD:C_0603_1608Metric"
 			(at 178.7652 107.95 0)
 			(effects
@@
 			)
 		)
-		(property "Footprint" ""
+		(property "Footprint" "Jumper:SolderJumper-2_P1.3mm_Open_RoundedPad1.0x1.5mm"
 			(at 118.11 106.68 0)
 			(effects
@@
 			)
 		)
-		(property "Footprint" ""
+		(property "Footprint" "Jumper:SolderJumper-2_P1.3mm_Open_RoundedPad1.0x1.5mm"
 			(at 125.73 106.68 0)
 			(effects
@@
 			)
 		)
-		(property "Footprint" ""
+		(property "Footprint" "Resistor_SMD:R_0603_1608Metric"
 			(at 198.882 99.06 90)
 			(effects
@@
 			)
 		)
-		(property "Footprint" ""
+		(property "Footprint" "Jumper:SolderJumper-2_P1.3mm_Open_RoundedPad1.0x1.5mm"
 			(at 121.92 106.68 0)
 			(effects
@@
 			)
 		)
-		(property "Footprint" ""
+		(property "Footprint" "Resistor_SMD:R_0603_1608Metric"
 			(at 110.49 103.378 90)
 			(effects
@@
 			)
 		)
-		(property "Footprint" ""
+		(property "Footprint" "Resistor_SMD:R_0603_1608Metric"
 			(at 115.57 100.838 90)
 			(effects
@@
 			)
 		)
-		(property "Footprint" ""
+		(property "Footprint" "Capacitor_SMD:C_0603_1608Metric"
 			(at 166.0652 107.95 0)
 			(effects
@@
 			)
 		)
-		(property "Footprint" ""
+		(property "Footprint" "Capacitor_SMD:C_0603_1608Metric"
 			(at 194.6148 102.87 0)
 			(effects

Commit message: Commit
Parts:
- removed JP2, JP3, JP4: SolderJumper_2_Open, Jumper:SolderJumper-2_P1.3mm_Open_RoundedPad1.0x1.5mm, symbol Jumper:SolderJumper_2_Open
- removed R34, R35: 10k, Resistor_SMD:R_0603_1608Metric, symbol Device:R
- D1: footprint (none) -> Diode_SMD:D_SOD-123
- D4: footprint Diode_THT:D_DO-41_SOD81_P10.16mm_Horizontal -> Diode_SMD:D_SOD-123
- T1: footprint IRF9310TRPBF:SO-8 -> Riqi_Parts:SO-8
Connections:
- net GND: now also U6.4 (A1), U6.9 (A2)
