File: Kicad/NIVARA/RELAY_INTERFACE.kicad_sch (KiCad schematic)
At the start: 3 parts, among them K1 G2RL-1, K2 G2RL-1

Commit message: ZZZ
Parts:
- removed U4: ~, Riqi_Parts:SOIC127P600X172-14N, symbol Riqi_Parts:BTS723GW
- added D1, D2: 1N4001, Diode_SMD:D_SMA, symbol Diode:1N4001
- added Q1, Q2: NCV8402xST, Package_TO_SOT_SMD:SOT-223, symbol Driver_FET:NCV8402xST
Connections:
- net GND: now also Q1.3 (S), Q2.3 (S); no longer K1.A2, K2.A2
- net RL1_EN: now also Q1.1 (G)
- net RL2_EN: now also Q2.1 (G)
- net VCC: now also K1.A1, K2.A1, D1.1 (K), D2.1 (K)
- new net: D1.2 (A), K1.A2, Q1.2 (D), Q1.4 (D)
- new net: D2.2 (A), K2.A2, Q2.2 (D), Q2.4 (D)
Other:
- moved on the sheet: K2

Commit message: .
Parts:
- removed D1, D2: 1N4001, Diode_SMD:D_SMA, symbol Diode:1N4001
- removed Q1, Q2: NCV8402xST, Package_TO_SOT_SMD:SOT-223, symbol Driver_FET:NCV8402xST
- added Q2: ~, symbol Riqi_Parts:LANKE LK1802
Connections:
- net GND: now also Q2.2 (E)
- net RL1_EN: now also Q2.3 (1B)
- net RL2_EN: now also Q2.4 (2B)
- net VCC: now also Q2.5 (COM)
- net at K1.A2: now also Q2.1 (1C)
- net at K2.A2: now also Q2.6 (2C)
Other:
- moved on the sheet: K1, K2

Commit message: Debí de enrutar antes :C
tengo sueño
Parts:
- Q2: footprint (none) -> Package_TO_SOT_SMD:SOT-363_SC-70-6
Changed lines of the file:
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@@
 			)
 		)
-		(property "Footprint" ""
+		(property "Footprint" "Package_TO_SOT_SMD:SOT-363_SC-70-6"
 			(at 105.41 105.41 0)
 			(effects

Commit message: Commit
Parts:
- removed K1, K2: G2RL-1, Relay_THT:Relay_SPDT_Omron_G2RL-1, symbol Relay:G2RL-1
Changed lines of the file:
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@@
-	)
-	(symbol
-		(lib_id "Relay:G2RL-1")
-		(at 125.73 97.79 0)
-		(unit 1)
-		(exclude_from_sim no)
-		(in_bom yes)
-		(on_board yes)
-		(dnp no)
-		(fields_autoplaced yes)
-		(property "Reference" "K1"
-			(at 137.16 96.5199 0)
-			(effects
-				(font
-					(size 1.27 1.27)
-				)
-				(justify left)
-			)
-		)
-		(property "Value" "G2RL-1"
-			(at 137.16 99.0599 0)
-			(effects
-				(font
-					(size 1.27 1.27)
-				)
-				(justify left)
-			)
-		)
-		(property "Footprint" "Relay_THT:Relay_SPDT_Omron_G2RL-1"
-			(at 137.16 99.06 0)
-			(effects
-				(font
-					(size 1.27 1.27)
-				)
-				(justify left)
-				(hide yes)
-			)
-		)
-		(property "Datasheet" "https://omronfs.omron.com/en_US/ecb/products/pdf/en-g2rl.pdf"
-			(at 125.73 97.79 0)
-			(effects
-				(font
-					(size 1.27 1.27)
-				)
-				(hide yes)
-			)
-		)
-		(property "Description" "General Purpose Low Profile Relay SPDT Through Hole, Omron G2RL series, 12A 250VAC"
-			(at 125.73 97.79 0)
-			(effects
-				(font
-					(size 1.27 1.27)
-				)
-				(hide yes)
-			)
-		)
-		(pin "14"
-		)
-		(pin "12"
-		)
-		(pin "A2"
-		)
-		(pin "11"
-		)
-		(pin "A1"
-		)
-		(instances
-			(project ""
-				(path "/8290cc18-06d0-4e02-a781-29a61ebc321a/9e4d7a0c-a5eb-4e88-9036-0c35e68b279a/86b88fb6-54fe-4cca-9b3c-121214f029ac"
-					(reference "K1")
-					(unit 1)
-				)
-			)
-		)
 	)
 	(symbol
@@
 					(unit 1)
 				)
-			)
-		)
-	)
-	(symbol
-		(lib_id "Relay:G2RL-1")
-		(at 167.64 99.06 0)
-		(unit 1)
-		(exclude_from_sim no)
-		(in_bom yes)
-		(on_board yes)
-		(dnp no)
-		(fields_autoplaced yes)
-		(property "Reference" "K2"
-			(at 179.07 97.7899 0)
-			(effects
-				(font
-					(size 1.27 1.27)
-				)
-				(justify left)
-			)
-		)
-		(property "Value" "G2RL-1"
-			(at 179.07 100.3299 0)
-			(effects
-				(font
-					(size 1.27 1.27)
-				)
-				(justify left)
-			)
-		)
-		(property "Footprint" "Relay_THT:Relay_SPDT_Omron_G2RL-1"
-			(at 179.07 100.33 0)
-			(effects
-				(font
-					(size 1.27 1.27)
-				)
-				(justify left)
-				(hide yes)
-			)
-		)
-		(property "Datasheet" "https://omronfs.omron.com/en_US/ecb/products/pdf/en-g2rl.pdf"
-			(at 167.64 99.06 0)
-			(effects
-				(font
-					(size 1.27 1.27)
-				)
-				(hide yes)
-			)
-		)
-		(property "Description" "General Purpose Low Profile Relay SPDT Through Hole, Omron G2RL series, 12A 250VAC"
-			(at 167.64 99.06 0)
-			(effects
-				(font
-					(size 1.27 1.27)
-				)
-				(hide yes)
-			)
-		)
-		(pin "14"
-		)
-		(pin "12"
-		)
-		(pin "A2"
-		)
-		(pin "11"
-		)
-		(pin "A1"
-		)
-		(instances
-			(project "NIVARA"
-				(path "/8290cc18-06d0-4e02-a781-29a61ebc321a/9e4d7a0c-a5eb-4e88-9036-0c35e68b279a/86b88fb6-54fe-4cca-9b3c-121214f029ac"
-					(reference "K2")
-					(unit 1)
-				)

Commit message: Faltan dos Cositas
Casi terminamos de enrutar
Parts:
- added K1, K2: TQ2-24V, Riqi_Parts:TQ2=24V, symbol Riqi_Parts:TQ2-24V
Connections:
- net RL1_COM: now also K1.3, K1.8
- net RL1_OUTPUT_NC: now also K1.2, K1.9
- net RL1_OUTPUT_NO: now also K1.4, K1.7
- net RL2_COM: now also K2.3, K2.8
- net RL2_OUTPUT_NC: now also K2.2, K2.9
- net RL2_OUTPUT_NO: now also K2.4, K2.7
- net VCC: now also K1.1, K2.1
- net at Q2.1 (1C): now also K1.10
- net at Q2.6 (2C): now also K2.10
