File: Kicad/NIVARA/NIVARA.kicad_pcb (KiCad board)
At the start: 2 copper layers, 7 parts, among them K1 G2RL-1, K2 G2RL-1, U1 ESP32-S3-WROOM-1, U2 AP63203WU

Commit message: tengo sueño
Hay que dormir
Parts:
- added D2: SM712_SOT23, Package_TO_SOT_SMD:SOT-23, F.Cu at (199.3, 88.3)
- added D3: SMF24A, Diode_SMD:D_SMF, F.Cu at (196.8, 121.0)
- added D4: 1N4007, Diode_THT:D_DO-41_SOD81_P10.16mm_Horizontal, F.Cu at (166.9, 88.0)
- added D5: SMF24A, Diode_SMD:D_SMF, F.Cu at (168.0, 98.5)
- added D6: SMF24A, Diode_SMD:D_SMF, F.Cu at (183.9, 113.9)
- added D7: SMF24A, Diode_SMD:D_SMF, F.Cu at (183.9, 117.2)
- added R10: 910, Resistor_SMD:R_0603_1608Metric, F.Cu at (176.9, 116.0)
- added R12: 910, Resistor_SMD:R_0603_1608Metric, F.Cu at (176.9, 118.6)
- added R18: 910, Resistor_SMD:R_0603_1608Metric, F.Cu at (176.9, 103.4)
- added R19: 910, Resistor_SMD:R_0603_1608Metric, F.Cu at (176.9, 105.9)
- added R36: 910, Resistor_SMD:R_0603_1608Metric, F.Cu at (192.8, 89.7)
- added R7: 910, Resistor_SMD:R_0603_1608Metric, F.Cu at (192.8, 87.1)
- added REF**: MountingHole_3.2mm_M3_DIN965_Pad, MountingHole:MountingHole_3.2mm_M3_DIN965_Pad, F.Cu at (129.7, 47.8)
- added REF**: MountingHole_3.2mm_M3_DIN965_Pad, MountingHole:MountingHole_3.2mm_M3_DIN965_Pad, F.Cu at (44.6, 97.8)
- added U10: LTV-357TB, Package_SO:SO-4_4.4x3.6mm_P2.54mm, F.Cu at (170.0, 110.2)
- added U11: ~, Riqi_Parts:eSOP-8, F.Cu at (197.8, 113.0)
- added U12: ~, Package_SO:SO-4_4.4x4.3mm_P2.54mm, F.Cu at (185.3, 107.3)
- added U13: ~, Package_SO:SO-4_4.4x4.3mm_P2.54mm, F.Cu at (196.1, 101.4)
- added U14: ~, Package_SO:SO-4_4.4x4.3mm_P2.54mm, F.Cu at (196.1, 107.3)
- added U15: LTV-357TB, Package_SO:SO-4_4.4x3.6mm_P2.54mm, F.Cu at (185.9, 93.9)
- added U2: AP63200WU, Package_TO_SOT_SMD:TSOT-23-6, F.Cu at (189.3, 114.6)
- added U4: LTV-357TB, Package_SO:SO-4_4.4x3.6mm_P2.54mm, F.Cu at (185.9, 88.6)
- added U5: ~, Package_SO:SO-4_4.4x4.3mm_P2.54mm, F.Cu at (185.3, 101.4)
- added U6: ~, Package_SO:SSOP-10-1EP_3.9x4.9mm_P1mm_EP2.1x3.3mm, F.Cu at (169.3, 93.6)
- added U7: LTV-357TB, Package_SO:SO-4_4.4x3.6mm_P2.54mm, F.Cu at (170.0, 117.5)
- added U8: LTV-357TB, Package_SO:SO-4_4.4x3.6mm_P2.54mm, F.Cu at (170.0, 122.8)
- added U9: LTV-357TB, Package_SO:SO-4_4.4x3.6mm_P2.54mm, F.Cu at (170.0, 104.9)
- moved JP1 88.4 mm to (230.3, 72.3)
- moved U1 88.4 mm to (214.8, 52.8)
- moved U2 88.4 mm to (230.7, 68.3)
- moved U3 88.4 mm to (205.9, 83.0)
- moved U4 88.4 mm to (271.9, 40.5)
- moved K2 88.4 mm to (256.0, 38.6)
- moved K1 84.8 mm to (238.2, 39.2)
Connections:
- net /NIVARA_BOARD/RS485_A renamed Net-(U3-A)
- net /NIVARA_BOARD/RS485_B renamed Net-(U3-B)
- JP1 pad 1: Net-(JP1-A) -> Net-(D6-A1)
- K1 pad A1: Net-(K1-PadA1) -> VCC
- K1 pad A2: GND -> Net-(Q2-1C)
- K2 pad A1: Net-(K2-PadA1) -> VCC
- K2 pad A2: GND -> Net-(Q2-2C)
- U1 pad 12: unconnected-(U1-GPIO8/TOUCH8/ADC1_CH7/SUBSPICS1-Pad12) -> /NIVARA_BOARD/PNP_IN_Mod/NPN_Output0
- U1 pad 15: unconnected-(U1-GPIO3/TOUCH3/ADC1_CH2-Pad15) -> /NIVARA_BOARD/RELAY_INTERFACE/RL2_EN
- U1 pad 16: unconnected-(U1-GPIO46-Pad16) -> /NIVARA_BOARD/~{TRANSMIT}/RECEIVE
- U1 pad 17: unconnected-(U1-GPIO9/TOUCH9/ADC1_CH8/FSPIHD/SUBSPIHD-Pad17) -> /NIVARA_BOARD/PNP_IN_Mod/NPN_Output1
- U1 pad 18: unconnected-(U1-GPIO10/TOUCH10/ADC1_CH9/FSPICS0/FSPIIO4/SUBSPICS0-Pad18) -> /NIVARA_BOARD/DRY_INPUT_INTERFACE/DRY_OUT0
- U1 pad 23: unconnected-(U1-GPIO21-Pad23) -> /NIVARA_BOARD/DRY_INPUT_INTERFACE/DRY_OUT1
- U1 pad 24: unconnected-(U1-GPIO47/SPICLK_P/SUBSPICLK_P_DIFF-Pad24) -> /NIVARA_BOARD/RS485_INTERFACE/UART_TX
- U1 pad 25: unconnected-(U1-GPIO48/SPICLK_N/SUBSPICLK_N_DIFF-Pad25) -> /NIVARA_BOARD/RS485_INTERFACE/UART_RX
- U1 pad 26: unconnected-(U1-GPIO45-Pad26) -> /NIVARA_BOARD/NPN_OUT_INTERFACE/NPN_EN1
- U1 pad 28: unconnected-(U1-SPIIO6/GPIO35/FSPID/SUBSPID-Pad28) -> /NIVARA_BOARD/VOLTAGE_AOUT_INTERFACE/SEL
- U1 pad 29: unconnected-(U1-SPIIO7/GPIO36/FSPICLK/SUBSPICLK-Pad29) -> /NIVARA_BOARD/~{RUN}/STOP
- U1 pad 31: unconnected-(U1-GPIO38/FSPIWP/SUBSPIWP-Pad31) -> /NIVARA_BOARD/NPN_OUT_INTERFACE/NPN_EN0
- U1 pad 36: /NIVARA_BOARD/RS485_INTERFACE/UART_RX -> unconnected-(U1-U0RXD/GPIO44/CLK_OUT2-Pad36)
- U1 pad 37: /NIVARA_BOARD/RS485_INTERFACE/UART_TX -> unconnected-(U1-U0TXD/GPIO43/CLK_OUT1-Pad37)
- U1 pad 38: unconnected-(U1-GPIO2/TOUCH2/ADC1_CH1-Pad38) -> /NIVARA_BOARD/RELAY_INTERFACE/RL1_EN
- U1 pad 39: unconnected-(U1-GPIO1/TOUCH1/ADC1_CH0-Pad39) -> /NIVARA_BOARD/mA_AINPUT
- U1 pad 4: unconnected-(U1-GPIO4/TOUCH4/ADC1_CH3-Pad4) -> /NIVARA_BOARD/32V_AIN_INTERFACE/32V_ADC
- U1 pad 5: unconnected-(U1-GPIO5/TOUCH5/ADC1_CH4-Pad5) -> /NIVARA_BOARD/10V_AIN_INTERFACE/10V_ADC
- U1 pad 6: unconnected-(U1-GPIO6/TOUCH6/ADC1_CH5-Pad6) -> /NIVARA_BOARD/PNP_OUT_INTERFACE/PNP_EN0
- U1 pad 7: unconnected-(U1-GPIO7/TOUCH7/ADC1_CH6-Pad7) -> /NIVARA_BOARD/PNP_OUT_INTERFACE/PNP_EN1
- U1 pad 8: unconnected-(U1-GPIO15/U0RTS/ADC2_CH4/XTAL_32K_P-Pad8) -> /NIVARA_BOARD/VOLTAGE_AOUT_INTERFACE/SDA
- U1 pad 9: unconnected-(U1-GPIO16/U0CTS/ADC2_CH5/XTAL_32K_N-Pad9) -> /NIVARA_BOARD/VOLTAGE_AOUT_INTERFACE/SCLK
Other:
- board outline added: 101.2 x 80.8 mm

Commit message: Debí de enrutar antes :C
tengo sueño
Parts:
- removed the U2 at (230.7, 68.3)
- removed the U4 at (271.9, 40.5)
- added C1: 1uF, Capacitor_SMD:C_0603_1608Metric, F.Cu at (166.1, 36.9)
- added C10: 100nF, Capacitor_SMD:C_0603_1608Metric, F.Cu at (125.8, 72.8)
- added C11: 100nF, Capacitor_SMD:C_0603_1608Metric, F.Cu at (133.5, 100.5)
- added C12: 220pF, Capacitor_SMD:C_0603_1608Metric, F.Cu at (78.8, 44.2)
- added C13: 1uF, Capacitor_SMD:C_0603_1608Metric, F.Cu at (75.5, 44.0)
- added C14: 1uF, Capacitor_SMD:C_0603_1608Metric, F.Cu at (83.0, 48.2)
- added C15: 100nF, Capacitor_SMD:C_0603_1608Metric, F.Cu at (101.0, 60.0)
- added C2: 100nF, Capacitor_SMD:C_0603_1608Metric, F.Cu at (50.0, 83.9)
- added C3: 10uF, Capacitor_SMD:C_0603_1608Metric, F.Cu at (46.5, 89.4)
- added C4: 22uF, Capacitor_SMD:C_0603_1608Metric, F.Cu at (49.8, 89.4)
- added C5: 22uF, Capacitor_SMD:C_0603_1608Metric, F.Cu at (49.8, 90.9)
- added C6: 100pF, Capacitor_SMD:C_0603_1608Metric, F.Cu at (43.8, 82.6)
- added C7: 1uF, Capacitor_SMD:C_0603_1608Metric, F.Cu at (182.2, 36.9)
- added C8: 100nF, Capacitor_SMD:C_0603_1608Metric, F.Cu at (182.2, 39.4)
- added C9: 100nF, Capacitor_SMD:C_0603_1608Metric, F.Cu at (131.2, 73.8)
- added J1: Screw_Terminal_01x03, TerminalBlock_4Ucon:TerminalBlock_4Ucon_1x03_P3.50mm_Horizontal, F.Cu at (60.3, 109.0)
- added J11: Screw_Terminal_01x02, TerminalBlock_4Ucon:TerminalBlock_4Ucon_1x02_P3.50mm_Horizontal, F.Cu at (49.2, 109.0)
- added J12: Screw_Terminal_01x04, TerminalBlock_4Ucon:TerminalBlock_4Ucon_1x04_P3.50mm_Horizontal, F.Cu at (71.9, 37.5)
- added J2: Screw_Terminal_01x03, TerminalBlock_4Ucon:TerminalBlock_4Ucon_1x03_P3.50mm_Horizontal, F.Cu at (74.8, 109.0)
- added J3: Screw_Terminal_01x04, TerminalBlock_4Ucon:TerminalBlock_4Ucon_1x04_P3.50mm_Horizontal, F.Cu at (89.4, 109.0)
- added J4: Screw_Terminal_01x03, TerminalBlock_4Ucon:TerminalBlock_4Ucon_1x03_P3.50mm_Horizontal, F.Cu at (107.5, 109.0)
- added J5: Screw_Terminal_01x02, TerminalBlock_4Ucon:TerminalBlock_4Ucon_1x02_P3.50mm_Horizontal, F.Cu at (122.0, 109.0)
- added J6: Screw_Terminal_01x06, TerminalBlock_4Ucon:TerminalBlock_4Ucon_1x06_P3.50mm_Horizontal, F.Cu at (96.9, 37.5)
- added J7: Screw_Terminal_01x03, TerminalBlock_4Ucon:TerminalBlock_4Ucon_1x03_P3.50mm_Horizontal, F.Cu at (54.0, 37.5)
- added J8: Screw_Terminal_01x03, TerminalBlock_4Ucon:TerminalBlock_4Ucon_1x03_P3.50mm_Horizontal, F.Cu at (111.3, 37.5)
- added J9: Screw_Terminal_01x03, TerminalBlock_4Ucon:TerminalBlock_4Ucon_1x03_P3.50mm_Horizontal, F.Cu at (125.8, 37.5)
- added L1: 6.8uH, Inductor_SMD:L_6.3x6.3_H3, F.Cu at (55.5, 84.9)
- added Q2: ~, Package_TO_SOT_SMD:SOT-363_SC-70-6, F.Cu at (152.0, 116.0)
- added R1: 10k, Resistor_SMD:R_0603_1608Metric, F.Cu at (166.1, 39.4)
- added R11: 412, Resistor_SMD:R_0603_1608Metric, F.Cu at (178.2, 61.0)
- added R13: 412, Resistor_SMD:R_0603_1608Metric, F.Cu at (178.2, 63.5)
- added R14: 160k, Resistor_SMD:R_0603_1608Metric, F.Cu at (131.2, 70.2)
- added R15: 13k, Resistor_SMD:R_0603_1608Metric, F.Cu at (131.2, 72.0)
- added R16: 51k, Resistor_SMD:R_0603_1608Metric, F.Cu at (125.8, 69.2)
- added R17: 16k, Resistor_SMD:R_0603_1608Metric, F.Cu at (125.8, 71.0)
- added R2: 196k, Resistor_SMD:R_0603_1608Metric, F.Cu at (45.5, 82.6)
- added R20: 412, Resistor_SMD:R_0603_1608Metric, F.Cu at (115.2, 75.2)
- added R21: 412, Resistor_SMD:R_0603_1608Metric, F.Cu at (114.2, 92.0)
- added R22: 10k, Resistor_SMD:R_0603_1608Metric, F.Cu at (166.1, 41.9)
- added R23: 10k, Resistor_SMD:R_0603_1608Metric, F.Cu at (182.2, 41.9)
- added R24: 120, Resistor_SMD:R_0603_1608Metric, F.Cu at (44.8, 54.8)
- added R25: 120, Resistor_SMD:R_0603_1608Metric, F.Cu at (44.8, 51.2)
- added R26: 100, Resistor_SMD:R_0603_1608Metric, F.Cu at (172.2, 63.5)
- added R27: 100k, Resistor_SMD:R_0603_1608Metric, F.Cu at (83.0, 46.5)
- added R28: 15, Resistor_SMD:R_0603_1608Metric, F.Cu at (105.0, 55.0)
- added R29: 100, Resistor_SMD:R_0603_1608Metric, F.Cu at (277.2, 125.0)
- added R3: 62k, Resistor_SMD:R_0603_1608Metric, F.Cu at (47.2, 82.6)
- added R30: 100, Resistor_SMD:R_0603_1608Metric, F.Cu at (277.2, 127.5)
- added R31: 4.7k, Resistor_SMD:R_0603_1608Metric, F.Cu at (166.1, 44.4)
- added R32: 4.7k, Resistor_SMD:R_0603_1608Metric, F.Cu at (166.1, 47.0)
- added R33: 10k, Resistor_SMD:R_0603_1608Metric, F.Cu at (77.2, 54.5)
- added R34: 10k, Resistor_SMD:R_0603_1608Metric, F.Cu at (105.0, 60.0)
- added R35: 10k, Resistor_SMD:R_0603_1608Metric, F.Cu at (105.0, 62.5)
- added R4: 100, Resistor_SMD:R_0603_1608Metric, F.Cu at (172.2, 61.0)
- added R5: 412, Resistor_SMD:R_0603_1608Metric, F.Cu at (115.8, 84.8)
- added R6: 2.5k, Resistor_SMD:R_0603_1608Metric, F.Cu at (78.8, 42.5)
- added R8: 120, Resistor_SMD:R_0603_1608Metric, F.Cu at (133.5, 98.8)
- added R9: 412, Resistor_SMD:R_0603_1608Metric, F.Cu at (115.8, 88.8)
- moved JP1 169.3 mm to (61.5, 85.1)
- moved D2 151.0 mm to (55.0, 43.8)
- moved U3 144.4 mm to (66.3, 46.3), turned to 180 degrees
- moved U2 144.1 mm to (48.0, 86.6)
- moved D7 144.0 mm to (42.2, 91.1), turned to 180 degrees
- moved D6 132.3 mm to (56.0, 80.1), turned to 180 degrees
- moved R7 129.9 mm to (64.0, 103.8)
- moved R36 129.3 mm to (63.8, 97.5)
- moved U4 122.7 mm to (63.8, 100.8), turned to 180 degrees
- moved U15 122.1 mm to (63.8, 94.2), turned to 180 degrees
- moved U6 102.3 mm to (77.2, 49.0), turned to 90 degrees
- moved R19 97.9 mm to (79.0, 104.0)
- moved R18 97.8 mm to (79.2, 97.2)
- moved U1 93.6 mm to (127.8, 87.2), turned to -90 degrees
- moved D5 92.3 mm to (85.9, 56.1)
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Connections:
- U1 pad 16: /NIVARA_BOARD/~{TRANSMIT}/RECEIVE -> /NIVARA_BOARD/RS485_INTERFACE/~{TX}/RX
- U1 pad 19: unconnected-(U1-GPIO11/TOUCH11/ADC2_CH0/FSPID/FSPIIO5/SUBSPID-Pad19) -> /NIVARA_BOARD/NPN_IN_Mod/NPN_Output0
- U1 pad 20: unconnected-(U1-GPIO12/TOUCH12/ADC2_CH1/FSPICLK/FSPIIO6/SUBSPICLK-Pad20) -> /NIVARA_BOARD/NPN_IN_Mod/NPN_Output1
- U6 pad 4: Net-(JP3-B) -> GND
- U6 pad 9: Net-(JP4-B) -> GND
Routing:
- net +3.3V: track 0.00 -> 122.9 mm, vias 0 -> 7
- net /NIVARA_BOARD/RS485_INTERFACE/UART_RX: track 0.00 -> 92.4 mm, vias 0 -> 2
- net /NIVARA_BOARD/RS485_INTERFACE/UART_TX: track 0.00 -> 90.3 mm, vias 0 -> 2
- net /NIVARA_BOARD/NPN_IN_Mod/NPN_Output1: track 0.00 -> 76.6 mm, vias 0 -> 2
- net /NIVARA_BOARD/RS485_INTERFACE/~{TX}/RX: track 0.00 -> 72.5 mm, vias 0 -> 3
- net /NIVARA_BOARD/+32V_AINPUT: track 0.00 -> 71.7 mm, vias 0 -> 3
- net /NIVARA_BOARD/+10V_AINPUT: track 0.00 -> 69.7 mm, vias 0 -> 3
- net /NIVARA_BOARD/NPN_IN_Mod/NPN_Output0: track 0.00 -> 67.8 mm, vias 0 -> 2
- net /NIVARA_BOARD/PNP_IN_Mod/NPN_Output0: track 0.00 -> 65.7 mm, vias 0 -> 2
- net /NIVARA_BOARD/PNP_IN_Mod/NPN_Output1: track 0.00 -> 57.3 mm, vias 0 -> 2
- net /NIVARA_BOARD/mA_AINPUT: track 0.00 -> 53.3 mm
- net Net-(D6-A1): track 0.00 -> 31.2 mm, vias 0 -> 2
- net GND: track 0.00 -> 30.4 mm, vias 0 -> 11
- net /NIVARA_BOARD/RS485_B: track 0.00 -> 30.0 mm, vias 0 -> 2
- net PNPIN_GND: track 0.00 -> 22.4 mm
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- added copper zone on F.Cu, net +3.3V
- added copper zone on F.Cu, net GND
- added copper zone on In1.Cu, net GND
- added copper zone on F.Cu, net Net-(D6-A1)
- added copper zone on F.Cu, net Net-(U2-SW)
- added copper zone on F.Cu, net VCC
Other:
- board size 101.2 x 80.8 mm -> 100.2 x 79.8 mm
- copper layers 2 -> 4

Commit message: Commit
Parts:
- removed R34, R35: 10k, Resistor_SMD:R_0603_1608Metric
- added D1: D_Zener, Diode_SMD:D_SOD-123, F.Cu at (61.8, 44.5)
- added T1: IRF9310TRPBF, Riqi_Parts:SO-8, F.Cu at (71.0, 47.8)
- D4: footprint Diode_THT:D_DO-41_SOD81_P10.16mm_Horizontal -> Diode_SMD:D_SOD-123
- K1, K2: value G2RL-1 -> SANYOU_SRD_Form_C; footprint Relay_THT:Relay_SPDT_Omron_G2RL-1 -> Relay_THT:Relay_SPDT_SANYOU_SRD_Series_Form_C
- moved K2 155.8 mm to (100.5, 47.8), turned to -90 degrees
- moved U11 132.8 mm to (81.2, 49.4), turned to 90 degrees
- moved D3 130.2 mm to (88.5, 48.8), turned to -90 degrees
- moved R29 129.9 mm to (184.0, 34.5)
- moved R30 129.9 mm to (184.0, 37.0)
- moved U13 129.9 mm to (180.5, 42.2)
- moved U14 129.9 mm to (180.5, 48.1)
- moved K1 121.9 mm to (117.5, 47.8), turned to -90 degrees
- moved C8 110.7 mm to (71.5, 42.8), turned to 180 degrees
- moved R23 98.4 mm to (83.8, 43.8), turned to 90 degrees
- moved C7 92.1 mm to (90.8, 48.0), turned to 90 degrees
- moved R28 34.8 mm to (70.2, 55.2), turned to 180 degrees
- moved D4 34.2 mm to (69.5, 53.2)
- moved Q2 32.1 mm to (165.2, 86.7)
- moved R10 32.1 mm to (190.1, 86.8)
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Connections:
- U11 pad 2: (no net) -> /NIVARA_BOARD/VOLTAGE_AOUT_INTERFACE/SDA
Routing:
- net /NIVARA_BOARD/VOLTAGE_AOUTPUT: track 0.00 -> 32.5 mm, vias 0 -> 1
- net /NIVARA_BOARD/mA_AOUTPUT+: track 0.00 -> 16.0 mm, vias 0 -> 1
- net Net-(U11-V5V): track 0.00 -> 14.4 mm
- net Net-(D5-A1): track 0.00 -> 12.5 mm
- net /NIVARA_BOARD/VOLTAGE_AOUT_INTERFACE/SDA: track 0.00 -> 10.9 mm, vias 0 -> 2
- net /NIVARA_BOARD/VOLTAGE_AOUT_INTERFACE/SCLK: track 0.00 -> 9.52 mm, vias 0 -> 2
- net Net-(U6-IOUT): track 0.00 -> 8.09 mm, vias 0 -> 2
- net Net-(D1-A): track 0.00 -> 5.89 mm
- net Net-(D4-A): track 0.00 -> 3.53 mm
- net /NIVARA_BOARD/VOLTAGE_AOUT_INTERFACE/SEL: track 0.00 -> 1.82 mm
- net /NIVARA_BOARD/+10V_AINPUT: track 69.7 -> 70.2 mm

Commit message: Faltan dos Cositas
Casi terminamos de enrutar
Parts:
- K1, K2: value SANYOU_SRD_Form_C -> TQ2-24V; footprint Relay_THT:Relay_SPDT_SANYOU_SRD_Series_Form_C -> Riqi_Parts:TQ2=24V
- moved R10 86.5 mm to (105.2, 103.5)
- moved R12 85.7 mm to (105.2, 101.8)
- moved R31 85.5 mm to (81.5, 56.2), turned to 90 degrees
- moved R32 83.4 mm to (83.3, 56.2), turned to 90 degrees
- moved R11 81.0 mm to (104.0, 93.5), turned to 180 degrees
- moved R13 79.4 mm to (104.0, 91.8), turned to 180 degrees
- moved U12 74.6 mm to (125.8, 61.6)
- moved U5 74.6 mm to (125.8, 55.8)
- moved R22 73.0 mm to (121.2, 99.5)
- moved U7 72.9 mm to (110.0, 98.8), turned to 90 degrees
- moved U8 69.1 mm to (114.2, 98.8), turned to 90 degrees
- moved Q2 68.5 mm to (102.0, 60.2), turned to 90 degrees
- moved R5 61.4 mm to (55.0, 93.5), turned to 180 degrees
- moved R9 59.9 mm to (56.2, 95.5), turned to 180 degrees
- moved R26 54.1 mm to (118.9, 53.9)
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Connections:
- J6 pad 2: /NIVARA_BOARD/RL1_OUTPUT_NC -> /NIVARA_BOARD/RL1_COM
- J6 pad 3: /NIVARA_BOARD/RL1_COM -> /NIVARA_BOARD/RL1_OUTPUT_NC
- J6 pad 5: /NIVARA_BOARD/RL2_OUTPUT_NC -> /NIVARA_BOARD/RL2_COM
- J6 pad 6: /NIVARA_BOARD/RL2_COM -> /NIVARA_BOARD/RL2_OUTPUT_NC
- K1 pad 1: /NIVARA_BOARD/RL2_COM -> VCC
- K1 pad 2: Net-(Q2-1C) -> /NIVARA_BOARD/RL1_OUTPUT_NC
- K1 pad 3: /NIVARA_BOARD/RL2_OUTPUT_NO -> /NIVARA_BOARD/RL1_COM
- K1 pad 4: /NIVARA_BOARD/RL2_OUTPUT_NC -> /NIVARA_BOARD/RL1_OUTPUT_NO
- K1 pad 5: VCC -> (no net)
- K2 pad 1: /NIVARA_BOARD/RL1_COM -> VCC
- K2 pad 2: Net-(Q2-2C) -> /NIVARA_BOARD/RL2_OUTPUT_NC
- K2 pad 3: /NIVARA_BOARD/RL1_OUTPUT_NO -> /NIVARA_BOARD/RL2_COM
- K2 pad 4: /NIVARA_BOARD/RL1_OUTPUT_NC -> /NIVARA_BOARD/RL2_OUTPUT_NO
- K2 pad 5: VCC -> (no net)
- R32 pad 2: /NIVARA_BOARD/VOLTAGE_AOUT_INTERFACE/SCLK -> /NIVARA_BOARD/VOLTAGE_AOUT_INTERFACE/SDA
Routing:
- net /NIVARA_BOARD/VOLTAGE_AOUT_INTERFACE/SCLK: track 9.52 -> 80.3 mm, vias 2 -> 4
- net /NIVARA_BOARD/VOLTAGE_AOUT_INTERFACE/SDA: track 10.9 -> 76.8 mm, vias 2 -> 4
- net /NIVARA_BOARD/RELAY_INTERFACE/RL1_EN: track 0.00 -> 65.4 mm, vias 0 -> 4
- net /NIVARA_BOARD/RL1_OUTPUT_NC: track 0.00 -> 42.5 mm
- net /NIVARA_BOARD/RELAY_INTERFACE/RL2_EN: track 0.00 -> 36.3 mm, vias 0 -> 4
- net /NIVARA_BOARD/RL2_OUTPUT_NO: track 0.00 -> 30.5 mm
- net /NIVARA_BOARD/RL2_OUTPUT_NC: track 0.00 -> 29.4 mm
- net /NIVARA_BOARD/RL1_COM: track 0.00 -> 26.2 mm
- net /NIVARA_BOARD/RL2_COM: track 0.00 -> 25.4 mm
- net /NIVARA_BOARD/DRY_INPUT_INTERFACE/DRY_OUT0: track 0.00 -> 23.4 mm, vias 0 -> 4
- net /NIVARA_BOARD/RL1_OUTPUT_NO: track 0.00 -> 21.8 mm
- net /NIVARA_BOARD/DRY_INPUT_INTERFACE/DRY_OUT1: track 0.00 -> 19.6 mm, vias 0 -> 2
- net VCC: track 21.8 -> 38.1 mm
- net /NIVARA_BOARD/~{RUN}/STOP: track 0.00 -> 13.0 mm
- net /NIVARA_BOARD/DRY_DINPUT_1: track 0.00 -> 10.8 mm
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
Commit message: ayuda
Parts:
- moved R29 24.3 mm to (126.5, 59.2)
- moved R30 20.5 mm to (126.8, 53.6)
- moved U12 16.8 mm to (116.2, 47.8), turned to 90 degrees
- moved U13 12.8 mm to (132.5, 60.5)
- moved U14 11.3 mm to (132.5, 55.0)
- moved U5 8.84 mm to (122.0, 47.8), turned to 90 degrees
- moved R26 3.92 mm to (115.0, 53.5), turned to 90 degrees
- moved R4 2.69 mm to (120.5, 53.5), turned to 90 degrees
Connections:
- U12 pad 3: /NIVARA_BOARD/NPN_DOUTPUT_0 -> /NIVARA_BOARD/NPN_DOUTPUT_1
Routing:
- net /NIVARA_BOARD/VOLTAGE_AOUT_INTERFACE/SEL: track 1.82 -> 87.6 mm, vias 0 -> 4
- net /NIVARA_BOARD/NPN_OUT_INTERFACE/NPN_EN1: track 0.00 -> 48.1 mm, vias 0 -> 2
- net /NIVARA_BOARD/NPN_OUT_INTERFACE/NPN_EN0: track 0.00 -> 44.3 mm, vias 0 -> 2
- net /NIVARA_BOARD/PNP_DOUTPUT_0: track 0.00 -> 36.1 mm
- net /NIVARA_BOARD/PNP_DOUTPUT_1: track 0.00 -> 29.2 mm
- net /NIVARA_BOARD/PNP_OUT_INTERFACE/PNP_EN1: track 0.00 -> 27.1 mm, vias 0 -> 2
- net /NIVARA_BOARD/NPN_DOUTPUT_0: track 0.00 -> 21.3 mm
- net /NIVARA_BOARD/PNP_OUT_INTERFACE/PNP_EN0: track 0.00 -> 20.9 mm, vias 0 -> 2
- net /NIVARA_BOARD/NPN_DOUTPUT_1: track 0.00 -> 17.9 mm
- net GND: track 30.4 -> 37.4 mm, vias 11 -> 17
- net Net-(R29-Pad2): track 0.00 -> 2.18 mm
- net Net-(R4-Pad2): track 0.00 -> 2.02 mm
- net Net-(R30-Pad2): track 0.00 -> 1.96 mm
- net Net-(R26-Pad2): track 0.00 -> 1.93 mm

Commit message: FINAL?
Routing:
- net +3.3V: track 126.6 -> 222.0 mm, vias 7 -> 17
- net GND: track 37.4 -> 71.9 mm, vias 17 -> 57
- net VCC: track 38.1 -> 47.1 mm, vias 0 -> 7
- added copper zone on In2.Cu, net +3.3V
- added copper zone on In2.Cu, net VCC
